Commit message: Odom to base_link and more MAGICgit status! (emoji de magia)

File: sim/ros2_ws/src/gmrai_description/urdf/GMR-AI.urdf (robot description, URDF)
Before this commit: robot GMR_AI, 7 links, 6 joints
Links:
- removed link robot_base
- added link base_link, mass 100.0; collision box size=1.000000 1.000000 0.200000; visual mesh filename=file:///home/adriangt2001/GMR-AI/sim/ros2_ws/src/gmrai_desc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
Joints:
- joint bl_joint: parent robot_base -> base_link
- joint br_joint: parent robot_base -> base_link
- joint fl_joint: parent robot_base -> base_link
- joint fr_joint: parent robot_base -> base_link
- joint tubo_joint: parent robot_base -> base_link
