Commit message: Changed vehicle weight

File: sim/ros2_ws/src/gmrai_description/urdf/GMR.urdf (robot description, URDF)
Before this commit: robot GMR_AI, 7 links, 6 joints
Links:
- link base_link: mass 100.0 -> 6.0
- link bl_link: mass 9.1891585117508 -> 0.5
- link br_link: mass 9.1891585117508 -> 0.5
- link cuchilla_link: mass 0.007853981633975 -> 0.01
- link fl_link: mass 9.1891585117508 -> 0.5
- link fr_link: mass 9.1891585117508 -> 0.5
- link tubo_link: mass 0.0314159265359 -> 0.01

Commit message: Added lidar and started with slam_toolbox

File: sim/ros2_ws/src/gmrai_description/urdf/GMR.urdf (robot description, URDF)
Before this commit: robot GMR_AI, 7 links, 6 joints
Links:
- added link lidar_link; collision cylinder length=0.01 radius=0.005; visual mesh filename=package://gmrai_description/urdf/GMR_body_vis_1.dae
- link base_link: geometry collision box size=1.000000 1.000000 0.200000; visual mesh filename=package://gmrai_description/urdf/GMR_base_vis_1.dae
- link bl_link: geometry collision cylinder length=0.13 radius=0.15; visual mesh filename=package://gmrai_description/urdf/GMR_llantas_ruedas_2_vis_1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
- link br_link: geometry collision cylinder length=0.13 radius=0.15; visual mesh filename=package://gmrai_description/urdf/GMR_llantas_ruedas_vis_1.d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
- link cuchilla_link: geometry collision mesh filename=package://gmrai_description/urdf/GMR_cuchilla_link_coll_1.d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; visual mesh filename=package://gmrai_description/urdf/GMR_cuchilla_vis_1.dae
- link fl_link: geometry collision cylinder length=0.13 radius=0.15; visual mesh filename=package://gmrai_description/urdf/GMR_llantas_ruedas_4_vis_1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
- link fr_link: geometry collision cylinder length=0.13 radius=0.15; visual mesh filename=package://gmrai_description/urdf/GMR_llantas_ruedas_3_vis_1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
- link tubo_link: geometry collision cylinder length=0.2288 radius=0.03; visual mesh filename=package://gmrai_description/urdf/GMR_tubo_vis_1.dae
Joints:
- added joint lidar_joint: type fixed, parent base_link, child lidar_link, origin xyz=0.000000 0.000000 0.200000 rpy=-3.141593 3.141593 -1.570796, axis 0 0 1

Commit message: Robot follows the path. Changed robot orientation (x axis forward)

File: sim/ros2_ws/src/gmrai_description/urdf/GMR.urdf (robot description, URDF)
Before this commit: robot GMR_AI, 8 links, 7 joints
Links:
- removed link lidar_link
- link base_link: geometry collision box size=1.000000 1.000000 0.200000; visual mesh filename=file:///home/adriangt2001/GMR-AI/sim/ros2_ws/src/gmrai_desc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
- link bl_link: geometry collision cylinder length=0.13 radius=0.15; visual mesh filename=file:///home/adriangt2001/GMR-AI/sim/ros2_ws/src/gmrai_desc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
- link br_link: geometry collision cylinder length=0.13 radius=0.15; visual mesh filename=file:///home/adriangt2001/GMR-AI/sim/ros2_ws/src/gmrai_desc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
- link cuchilla_link: geometry collision mesh filename=file:///home/adriangt2001/GMR-AI/sim/ros2_ws/src/gmrai_desc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; visual mesh filename=file:///home/adriangt2001/GMR-AI/sim/ros2_ws/src/gmrai_desc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
- link fl_link: geometry collision cylinder length=0.13 radius=0.15; visual mesh filename=file:///home/adriangt2001/GMR-AI/sim/ros2_ws/src/gmrai_desc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
- link fr_link: geometry collision cylinder length=0.13 radius=0.15; visual mesh filename=file:///home/adriangt2001/GMR-AI/sim/ros2_ws/src/gmrai_desc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
- link tubo_link: geometry collision cylinder length=0.2288 radius=0.03; visual mesh filename=file:///home/adriangt2001/GMR-AI/sim/ros2_ws/src/gmrai_desc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
Joints:
- removed joint lidar_joint
- joint bl_joint: origin xyz=-0.460000 -0.345000 -0.320000 rpy=3.141593 1.570796 0.000000 -> xyz=-0.355000 0.445000 -0.320000 rpy=-1.570796 1.570796 0.000000
- joint br_joint: origin xyz=0.431000 -0.345000 -0.320000 rpy=0.000000 1.570796 0.000000 -> xyz=-0.355000 -0.435000 -0.320000 rpy=1.570796 1.570796 0.000000
- joint fl_joint: origin xyz=-0.435000 0.345000 -0.320000 rpy=-3.141593 1.570796 0.000000 -> xyz=0.335000 0.430000 -0.320000 rpy=-1.570796 1.570796 0.000000
- joint fr_joint: origin xyz=0.431000 0.345000 -0.320000 rpy=0.000000 1.570796 0.000000 -> xyz=0.335000 -0.435000 -0.320000 rpy=1.570796 1.570796 0.000000

Commit message: More cleanup and generalization

File: sim/ros2_ws/src/gmrai_description/urdf/GMR.urdf (robot description, URDF)
Before this commit: robot GMR_AI, 7 links, 6 joints
Links:
- link base_link: geometry collision box size=1.000000 1.000000 0.200000; visual mesh filename=package://gmrai_description/urdf/GMR_base_vis_1.dae
- link bl_link: geometry collision cylinder length=0.13 radius=0.15; visual mesh filename=package://gmrai_description/urdf/GMR_llantas_ruedas_2_vis_1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
- link br_link: geometry collision cylinder length=0.13 radius=0.15; visual mesh filename=package://gmrai_description/urdf/GMR_llantas_ruedas_vis_1.d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
- link cuchilla_link: geometry collision mesh filename=package://gmrai_description/urdf/GMR_cuchilla_link_coll_1.d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; visual mesh filename=package://gmrai_description/urdf/GMR_cuchilla_vis_1.dae
- link fl_link: geometry collision cylinder length=0.13 radius=0.15; visual mesh filename=package://gmrai_description/urdf/GMR_llantas_ruedas_4_vis_1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
- link fr_link: geometry collision cylinder length=0.13 radius=0.15; visual mesh filename=package://gmrai_description/urdf/GMR_llantas_ruedas_3_vis_1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
- link tubo_link: geometry collision cylinder length=0.2288 radius=0.03; visual mesh filename=package://gmrai_description/urdf/GMR_tubo_vis_1.dae
